Commit message: 3

File: src/robot_description/urdf/target.urdf (robot description, URDF)
Before this commit: robot with_craw, 16 links, 15 joints
Links:
- removed link crawler_deap12_1
- added link cralwer_deap2_1, mass 0.2861324999999951; collision mesh filename=package://robot_description/meshes/cralwer_deap2_1.stl scale=0.001 0.001 0.001; visual mesh filename=package://robot_description/meshes/cralwer_deap2_1.stl scale=0.001 0.001 0.001
- link cralwer_deap_1: mass 0.23667750006845484 -> 0.28613249999999474
Joints:
- removed joint Slider 47
- removed joint Slider 49
- added joint Slider 52: type prismatic, parent craw_1, child cralwer_deap_1, origin xyz=0.009 -0.054 -0.00325 rpy=0 0 0, axis 1.0 -0.0 -0.0, limit lower=-0.01 upper=0.01 effort=100 velocity=100
- added joint Slider 53: type prismatic, parent craw_1, child cralwer_deap2_1, origin xyz=0.063 -0.054 -0.00325 rpy=0 0 0, axis 1.0 -0.0 -0.0, limit lower=-0.01 upper=0.01 effort=100 velocity=100

Commit message: A

File: src/robot_description/urdf/target.urdf (robot description, URDF)
Before this commit: robot with_craw, 16 links, 15 joints
Joints:
- removed joint Revolute 22
- added joint Revolute_22: type revolute, parent joint252_1, child 25joint_v2_1, origin xyz=0.0 -0.069999 0.076501 rpy=0 0 0, axis 0.0 -1.0 0.0, limit lower=-0.3491 upper=0.3491 effort=10 velocity=1.0

Commit message: AAAAA

File: src/robot_description/urdf/target.urdf (robot description, URDF)
Before this commit: robot with_craw, 16 links, 15 joints
Joints:
- joint Revolute_22: limit lower=-0.3491 upper=0.3491 effort=10 velocity=1.0 -> lower=-0.175 upper=0.175 effort=10 velocity=1.0

Commit message: D

File: src/robot_description/urdf/target.urdf (robot description, URDF)
Before this commit: robot with_craw, 16 links, 15 joints
Joints:
- joint Revolute_22: limit lower=-0.175 upper=0.175 effort=10 velocity=1.0 -> lower=-1.47 upper=1.47 effort=10 velocity=1.0
